File: kicad_SubBoards/SubBoards.kicad_pcb (KiCad board)
At the start: 2 copper layers, 7 parts, among them J1 Conn_01x10_Pin, J2 Conn_01x08_Pin, SW1 SW_Rotary_1x8_MP

Commit message: Completed subboards
Parts:
- removed RV1, RV2, RV3, RV4: R_Potentiometer_Small, Potentiometer_THT:Potentiometer_Alps_RK163_Single_Horizontal
- removed SW1: SW_Rotary_1x8_MP, Rotary_Encoder:RotaryEncoder_Alps_EC11E_Vertical_H20mm_CircularMountingHoles
- added S1: SR2612F-0112-21R0B-D8-N, SamacSys:SR2612F011221R0BD8N, F.Cu at (173.5, 86.8)
- added VR1: PTD904-2015Kc104, SamacSys:PTD9042015Kc104, F.Cu at (153.8, 100.6)
- moved J2 57.2 mm to (147.4, 80.4), turned to 0 degrees
- moved J1 12.5 mm to (172.7, 71.6)
Connections:
- J1 pad 10: Net-(J1-Pin_10) -> unconnected-(J1-Pin_10-Pad10)
Routing:
- net Net-(J1-Pin_8): track 0.00 -> 40.9 mm
- net Net-(J2-Pin_2): track 55.4 -> 22.8 mm
- net Net-(J2-Pin_1): track 52.3 -> 22.9 mm
- net Net-(J1-Pin_7): track 0.00 -> 25.5 mm
- net Net-(J2-Pin_5): track 34.1 -> 10.8 mm
- net Net-(J1-Pin_9): track 0.00 -> 20.9 mm
- net Net-(J1-Pin_6): track 0.00 -> 19.2 mm
- net Net-(J2-Pin_4): track 46.3 -> 27.1 mm
- net Net-(J1-Pin_1): track 0.00 -> 15.5 mm
- net Net-(J1-Pin_5): track 0.00 -> 15.0 mm
- net Net-(J2-Pin_6): track 27.6 -> 14.3 mm
- net Net-(J2-Pin_3): track 44.0 -> 31.2 mm
- net Net-(J1-Pin_4): track 0.00 -> 11.0 mm
- net Net-(J1-Pin_2): track 0.00 -> 10.7 mm
- net Net-(J2-Pin_8): track 13.6 -> 24.1 mm
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Other:
- board outline added: 54.9 x 39 mm
