File: kicad_SubBoards/SubBoards.kicad_sch (KiCad schematic)
At the start: 7 parts, among them J1 Conn_01x10_Pin, J2 Conn_01x08_Pin, SW1 SW_Rotary_1x8_MP

Commit message: Completed subboards
Parts:
- removed RV1, RV2, RV3, RV4: R_Potentiometer_Small, Potentiometer_THT:Potentiometer_Alps_RK163_Single_Horizontal, symbol Device:R_Potentiometer_Small
- removed SW1: SW_Rotary_1x8_MP, Rotary_Encoder:RotaryEncoder_Alps_EC11E_Vertical_H20mm_CircularMountingHoles, symbol Switch:SW_Rotary_1x8_MP
- added S1: SR2612F-0112-21R0B-D8-N, SamacSys:SR2612F011221R0BD8N, symbol SamacSys:SR2612F-0112-21R0B-D8-N
- added VR1: PTD904-2015Kc104, SamacSys:PTD9042015Kc104, symbol SamacSys:PTD904-2015Kc104
Connections:
- net at J2.3 (Pin_3): now also VR1.R13 (CW_1)
- net at J2.4 (Pin_4): now also VR1.R11 (CCW_1), VR1.R12 (WIPER_1)
- net at J2.1 (Pin_1): now also VR1.R21 (CCW_2), VR1.R22 (WIPER_2)
- net at J2.2 (Pin_2): now also VR1.R23 (CW_2)
- net at J2.5 (Pin_5): now also VR1.R43 (CW_4)
- net at J2.6 (Pin_6): now also VR1.R41 (CCW_4), VR1.R42 (WIPER_4)
- net at J1.1 (Pin_1): now also S1.1
- net at J1.2 (Pin_2): now also S1.2
- net at J1.3 (Pin_3): now also S1.3
- net at J1.4 (Pin_4): now also S1.4
- net at J1.5 (Pin_5): now also S1.5
- net at J1.6 (Pin_6): now also S1.6
- net at J1.7 (Pin_7): now also S1.7
- net at J1.8 (Pin_8): now also S1.8
- net at J1.9 (Pin_9): now also S1.A1
- net at J2.7 (Pin_7): now also VR1.R33 (CW_3)
- net at J2.8 (Pin_8): now also VR1.R31 (CCW_3), VR1.R32 (WIPER_3)
Other:
- moved on the sheet: J2
