File: kicad_SwitchBoard/SwitchBoard.kicad_pcb (KiCad board)
At the start: 2 copper layers, 47.8 x 37.6 mm, 20 parts, among them J1 Conn_01x04_Pin, J2 Conn_01x04_Pin, J3 Conn_01x03_Pin, SW1 SW_4PDT_x4

Commit message: Completed V1.0
Parts:
- added REF**: MountingHole_2.2mm_M2, MountingHole:MountingHole_2.2mm_M2, F.Cu at (141.8, 117.3)
- added REF**: MountingHole_2.2mm_M2, MountingHole:MountingHole_2.2mm_M2, F.Cu at (141.8, 86.8)
- SW1: footprint SamacSys:PBH4UEENAGVX -> ACRM:PushSwitch_4PDT_2x6Pin_P3.18x2.8
- moved SW1 5.39 mm to (136.1, 103.5)
- moved D1 1.62 mm to (141.9, 93.0)
Routing:
- net GND: track 87.8 -> 115.5 mm
- net Net-(D1-AK): track 28.5 -> 31.3 mm
- net Net-(J3-Pin_1): track 23.0 -> 25.5 mm
- net Net-(SW1C-B): track 40.2 -> 37.8 mm
- net Net-(SW1C-A): track 48.7 -> 46.4 mm
- net Net-(SW1C-C): track 31.8 -> 29.7 mm
- net Net-(J3-Pin_3): track 17.4 -> 19.3 mm
- net Net-(SW1A-A): track 48.5 -> 46.5 mm
- net Net-(SW1A-B): track 40.3 -> 38.6 mm
- net Net-(SW1A-C): track 32.0 -> 30.4 mm
- net Net-(D1-KA): track 42.3 -> 43.1 mm
Other:
- board size 47.8 x 37.6 mm -> 48 x 37.6 mm
- board text added: "- 0v +"
- board text added: "I1 I2 O G"
- board text added: "Polarity Sw"
- board text added: "Polarity Switch (AllPass Filter)"
- board text added: "V1.0, Andrew Martin, acramonics, June 2026"
