File: kicad_SwitchBoard/SwitchBoard.kicad_sch (KiCad schematic)
At the start: 20 parts, among them J1 Conn_01x04_Pin, J2 Conn_01x04_Pin, J3 Conn_01x03_Pin, SW1 SW_4PDT_x4

Commit message: Completed V1.0
Parts:
- SW1: footprint SamacSys:PBH4UEENAGVX -> ACRM:PushSwitch_4PDT_2x6Pin_P3.18x2.8
